Commit message: worked on tag to robot pose

File: robot_control/urdf/guy_robot.urdf (robot description, URDF)
Before this commit: robot robot, 23 links, 22 joints
Links:
- removed link camera_link
- added link camera; visual sphere radius=0.025
Joints:
- joint post_camera: child camera_link -> camera; origin xyz=0 0 0.031 rpy=0 0 0 -> xyz=0 0 0.031 rpy=-1.570796327 0 -1.570796327

Commit message: added pitch to URDF to tip robot back

File: robot_control/urdf/guy_robot.urdf (robot description, URDF)
Before this commit: robot robot, 23 links, 22 joints
Joints:
- joint base_footprint_link: origin xyz=-0.065 0 0.146 rpy=0 0 0 -> xyz=-0.065 0 0.146 rpy=0 0.04619 0
